File: PCB/Function/Function.kicad_pcb (KiCad board)
At the start: 2 copper layers, 101.6 x 152.4 mm, 141 parts, among them J1 MTA156-3, J2 MTA156-3-PWR, J3 MN12, J4 MN12, J5 MN12, J6 MBNF15, J7 MBNF15, Q1 BC847, Q2 BCM857, U1 AD823, U10 AD823, U11 ADG419, U12 4013, U15 ADR5045, U2 AD823, U3 AD823, U4 AD823, U5 AD823, U6 AD823, U7 AD823, U8 AD823, U9 AD823

Commit message: Update fn
Parts:
- moved C22 3.28 mm to (76.0, 162.0)
