File: PCB/Function/Function.kicad_sch (KiCad schematic)
At the start: 142 parts, among them J1 MTA156-3, J2 MTA156-3-PWR, J3 MN12, J4 MN12, J5 MN12, J6 MBNF15, J7 MBNF15, Q1 BC847, Q2 BCM857, U1 AD823, U10 AD823, U11 ADG419, U12 4013, U15 ADR5045, U2 AD823, U3 AD823, U4 AD823, U5 AD823, U6 AD823, U7 AD823, U8 AD823, U9 AD823

Commit message: Update fn
Connections:
- net GND: now also R21.1, R24.1; no longer U12.3 (C), U12.4 (R)
- net LIM: now also U12.4 (R)
- net LP: no longer R21.1, R24.1
- net TRIG: now also U12.3 (C)
- net at R12.1, R13.2: now also U2.5 (+); no longer U2.6 (-)
- net at R16.1, R17.2: now also U2.6 (-); no longer U2.5 (+)
